Commit message: robot model fix's baseline

File: test_7_description/test_7_description/urdf/test_7.urdf (robot description, URDF)
Before this commit: robot test_7, 25 links, 24 joints
Joints:
- joint Revolute 17: axis 1.0 0.0 0.0 -> 1.0 -0.0 0.0
- joint Revolute 18: axis 0.0 0.0 -1.0 -> 0.0 -0.0 -1.0
- joint Revolute 21: axis 1.0 0.0 0.0 -> -1.0 0.0 -0.0
- joint Revolute 22: axis 1.0 0.0 0.0 -> -1.0 0.0 -0.0
- joint Revolute 23: axis 0.0 0.0 -1.0 -> 0.0 -0.0 -1.0
- joint Revolute 24: axis 0.0 0.0 -1.0 -> 0.0 -0.0 -1.0
- joint Revolute 25: axis 0.0 0.0 -1.0 -> -0.0 0.0 1.0
- joint Revolute 26: axis 0.0 0.0 -1.0 -> -0.0 0.0 1.0
- joint Revolute 27: axis 0.0 0.0 -1.0 -> -0.0 0.0 1.0

File: test_7_description/test_7_description/urdf/test_7.xacro (robot description, xacro)
@@ -446,5 +446,5 @@
 <link name="left_feet_3">
   <inertial>
-    <origin xyz="-0.056770902465522896 -0.06389571088452764 0.003535511319261171" rpy="0 0 0"/>
+    <origin xyz="-0.05677090246552301 -0.06389571088452771 0.003535511319261206" rpy="0 0 0"/>
     <mass value="0.05603663809191365"/>
     <inertia ixx="0.000134" iyy="2.8e-05" izz="0.000156" ixy="-2.6e-05" iyz="0.0" ixz="-0.0"/>
@@ -466,5 +466,5 @@
 <link name="left_feet_2">
   <inertial>
-    <origin xyz="-0.05677090246552303 -0.06389571088452778 0.0035355113192612198" rpy="0 0 0"/>
+    <origin xyz="-0.056770902465523035 -0.06389571088452775 0.0035355113192611365" rpy="0 0 0"/>
     <mass value="0.05603663809191365"/>
     <inertia ixx="0.000134" iyy="2.8e-05" izz="0.000156" ixy="-2.6e-05" iyz="0.0" ixz="-0.0"/>
@@ -486,5 +486,5 @@
 <link name="left_feet_1">
   <inertial>
-    <origin xyz="-0.05677090246552319 -0.06389571088452783 0.0035353558362659562" rpy="0 0 0"/>
+    <origin xyz="-0.056770902465523104 -0.06389571088452775 0.0035353558362659562" rpy="0 0 0"/>
     <mass value="0.05603663809191365"/>
     <inertia ixx="0.000134" iyy="2.8e-05" izz="0.000156" ixy="-2.6e-05" iyz="0.0" ixz="-0.0"/>
@@ -582,5 +582,5 @@
   <parent link="top_bottom_connector_5"/>
   <child link="motor_holder_5"/>
-  <axis xyz="1.0 0.0 0.0"/>
+  <axis xyz="1.0 -0.0 0.0"/>
 </joint>
 <joint name="Revolute 18" type="continuous">
@@ -588,5 +588,5 @@
   <parent link="motor_holder_5"/>
   <child link="left_feet_connect_5"/>
-  <axis xyz="0.0 0.0 -1.0"/>
+  <axis xyz="0.0 -0.0 -1.0"/>
 </joint>
 <joint name="Rigid 19" type="fixed">
@@ -604,5 +604,5 @@
   <parent link="top_bottom_connector_7"/>
   <child link="motor_holder_7"/>
-  <axis xyz="1.0 0.0 0.0"/>
+  <axis xyz="-1.0 0.0 -0.0"/>
 </joint>
 <joint name="Revolute 22" type="continuous">
@@ -610,5 +610,5 @@
   <parent link="top_bottom_connector_6"/>
   <child link="motor_holder_6"/>
-  <axis xyz="1.0 0.0 0.0"/>
+  <axis xyz="-1.0 0.0 -0.0"/>
 </joint>
 <joint name="Revolute 23" type="continuous">
@@ -616,5 +616,5 @@
   <parent link="motor_holder_6"/>
   <child link="left_feet_connect_6"/>
-  <axis xyz="0.0 0.0 -1.0"/>
+  <axis xyz="0.0 -0.0 -1.0"/>
 </joint>
 <joint name="Revolute 24" type="continuous">
@@ -622,5 +622,5 @@
   <parent link="motor_holder_7"/>
   <child link="left_feet_connect_4"/>
-  <axis xyz="0.0 0.0 -1.0"/>
+  <axis xyz="0.0 -0.0 -1.0"/>
 </joint>
 <joint name="Revolute 25" type="continuous">
@@ -628,5 +628,5 @@
   <parent link="left_feet_connect_5"/>
   <child link="left_feet_3"/>
-  <axis xyz="0.0 0.0 -1.0"/>
+  <axis xyz="-0.0 0.0 1.0"/>
 </joint>
 <joint name="Revolute 26" type="continuous">
@@ -634,5 +634,5 @@
   <parent link="left_feet_connect_6"/>
   <child link="left_feet_2"/>
-  <axis xyz="0.0 0.0 -1.0"/>
+  <axis xyz="-0.0 0.0 1.0"/>
 </joint>
 <joint name="Revolute 27" type="continuous">
@@ -640,5 +640,5 @@
   <parent link="left_feet_connect_4"/>
   <child link="left_feet_1"/>
-  <axis xyz="0.0 0.0 -1.0"/>
+  <axis xyz="-0.0 0.0 1.0"/>
 </joint>
 </robot>
